File: hardware/schematics/data/piano_keys.brd (EAGLE design)
At the start: 148.1 x 15.2 mm, 14 parts

Commit message: adjusted key distances
Parts:
- moved LED4 5.00 mm to (42.0, 5.00)
- moved LED9 2.50 mm to (108.5, 5.00)
- moved SV1 0.19 mm to (6.60, 11.8)
- moved SV2 0.11 mm to (141.0, 12.0)
Connections:
- removed net DOUT: LED12.2-DOUT, SV1.2, SV2.3
- new net DIN_1: SV1.2, SV2.2
- new net DOUT_1: LED12.2-DOUT, SV2.3
Routing:
- net DOUT: track 146.7 -> 0.00 mm, vias 1 -> 0
- net DIN_1: track 0.00 -> 133.7 mm, vias 0 -> 1
- net 5V1: track 184.0 -> 296.7 mm
- net DOUT_1: track 0.00 -> 17.2 mm
- net GND: track 156.2 -> 162.7 mm
- net N$2: track 7.72 -> 12.7 mm
- net N$3: track 12.7 -> 7.73 mm
- net N$8: track 12.7 -> 10.2 mm
- net N$7: track 7.73 -> 10.2 mm
- added copper zone on layer 16, net N$1
- removed copper zone on layer 1, net N$1
Other:
- board size 148.1 x 15.2 mm -> 148 x 15 mm
