File: hardware/combined/combined.brd (EAGLE design)
At the start: 43.2 x 86 mm, 90 parts, among them Q1 CMA-4544PF-W, Q2 40M, U3 TCA9535PWR, U4 CSD18532Q5B_DNK_8, U5 CSD18532Q5B_DNK_8, U6 TPS62152_RGT_16, U7 CD4532B_NS_16, U8 TPS62152_RGT_16, X1 52745-2490, X2 32.768

Commit message: final board 1
Parts:
- added C6, C8: (no value), resistor:C0805K
- added D3: (no value), adafruit:SOD-323F
- added L3: (no value), inductor-neosid:MS85
- U$6, U$7: device power_module:DNK8 -> power_module:MP04A
- moved R10 88.4 mm to (8.89, 10.2), turned to 180 degrees
- moved R24 49.5 mm to (15.2, 15.2)
- moved R11 47.8 mm to (12.7, 25.4), turned to 180 degrees
- moved U$6 1.80 mm to (14.0, 48.3), turned to 0 degrees
- moved U$7 1.80 mm to (33.0, 48.3), turned to 0 degrees
- moved C4 1.27 mm to (11.4, 15.2)
- moved U3 1.27 mm to (6.35, 20.3)
- moved U7 1.27 mm to (36.8, 20.3)
- turned R22 to 90 degrees
Connections:
- new net L1OUT: C6.1, C8.1, L3.2, PACK+.15, R11.1
- net CHGOUT: now also D3.C, L3.1; no longer PACK+.15, R11.1
- net GND: now also C6.2, C8.2, D3.A
