File: hardware/combined/combined.sch (EAGLE design)
At the start: 90 parts, among them Q1 CMA-4544PF-W, Q2 40M, U3 TCA9535PWR, U4 CSD18532Q5B_DNK_8, U5 CSD18532Q5B_DNK_8, U6 TPS62152_RGT_16, U7 CD4532B_NS_16, U8 TPS62152_RGT_16, X1 52745-2490, X2 32.768

Commit message: final board 1
Parts:
- added C6, C8: (no value), resistor:C-USC0805K
- added D3: (no value), adafruit:DIODESOD-323F
- added L3: (no value), inductor-neosid:MS85
Connections:
- new net L1OUT: C6.1, C8.1, L3.2, PACK+.SNS, R11.1
- net CHGOUT: now also D3.C, L3.1; no longer PACK+.SNS, R11.1
- net GND: now also C6.2, C8.2, D3.A
Changed lines of the file:
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@@
 <part name="SV3" library="con-lstb" library_urn="urn:adsk.eagle:library:162" deviceset="MA04-1" device="" package3d_urn="urn:adsk.eagle:package:8337/1"/>
 <part name="SV4" library="con-lstb" library_urn="urn:adsk.eagle:library:162" deviceset="MA04-1" device="" package3d_urn="urn:adsk.eagle:package:8337/1"/>
+<part name="L3" library="inductor-neosid" library_urn="urn:adsk.eagle:library:241" deviceset="MS85" device="" package3d_urn="urn:adsk.eagle:package:14698/1"/>
+<part name="C6" library="resistor" library_urn="urn:adsk.eagle:library:348" deviceset="C-US" device="C0805K" package3d_urn="urn:adsk.eagle:package:26201/1"/>
+<part name="GND3" library="supply1" library_urn="urn:adsk.eagle:library:371" deviceset="GND" device=""/>
+<part name="C8" library="resistor" library_urn="urn:adsk.eagle:library:348" deviceset="C-US" device="C0805K" package3d_urn="urn:adsk.eagle:package:26201/1"/>
+<part name="D3" library="adafruit" library_urn="urn:adsk.eagle:library:420" deviceset="DIODE" device="SOD-323F"/>
 </parts>
 <sheets>
@@
 <instance part="C4" gate="G$1" x="40.64" y="20.32"/>
 <instance part="SV2" gate="G$1" x="58.42" y="-20.32"/>
+<instance part="L3" gate="G$1" x="73.66" y="45.72"/>
+<instance part="C6" gate="G$1" x="81.28" y="43.18"/>
+<instance part="GND3" gate="1" x="81.28" y="35.56"/>
+<instance part="C8" gate="G$1" x="86.36" y="43.18"/>
+<instance part="D3" gate="G$1" x="68.58" y="40.64" rot="R90"/>
 </instances>
 <busses>
@@
 <label x="71.12" y="-22.86" size="1.778" layer="95"/>
 </segment>
+<segment>
+<pinref part="C6" gate="G$1" pin="2"/>
+<pinref part="GND3" gate="1" pin="GND"/>
+<pinref part="C8" gate="G$1" pin="2"/>
+<wire x1="81.28" y1="38.1" x2="86.36" y2="38.1" width="0.1524" layer="91"/>
+<junction x="81.28" y="38.1"/>
+<pinref part="D3" gate="G$1" pin="A"/>
+<wire x1="68.58" y1="38.1" x2="81.28" y2="38.1" width="0.1524" layer="91"/>
+</segment>
 </net>
 <net name="PACK" class="0">
@@
 </segment>
 <segment>
-<pinref part="R11" gate="G$1" pin="1"/>
-<wire x1="20.32" y1="5.08" x2="10.16" y2="5.08" width="0.1524" layer="91"/>
-<label x="10.16" y="5.08" size="1.778" layer="95"/>
-</segment>
-<segment>
-<pinref part="PACK+" gate="A" pin="SNS"/>
-<wire x1="40.64" y1="33.02" x2="88.9" y2="33.02" width="0.1524" layer="91"/>
+<pinref part="L3" gate="G$1" pin="1"/>
 <pinref part="PACK+" gate="A" pin="OUT"/>
-<wire x1="40.64" y1="45.72" x2="88.9" y2="45.72" width="0.1524" layer="91"/>
+<wire x1="40.64" y1="45.72" x2="68.58" y2="45.72" width="0.1524" layer="91"/>
 <label x="48.26" y="45.72" size="1.778" layer="95"/>
-<wire x1="88.9" y1="45.72" x2="53.34" y2="45.72" width="0.1524" layer="91"/>
-<wire x1="88.9" y1="33.02" x2="88.9" y2="45.72" width="0.1524" layer="91"/>
-<junction x="88.9" y="45.72"/>
+<pinref part="D3" gate="G$1" pin="C"/>
+<wire x1="68.58" y1="43.18" x2="68.58" y2="45.72" width="0.1524" layer="91"/>
+<junction x="68.58" y="45.72"/>
 </segment>
 </net>
@@
 </segment>
 </net>
+<net name="L1OUT" class="0">
+<segment>
+<pinref part="R11" gate="G$1" pin="1"/>
+<wire x1="20.32" y1="5.08" x2="10.16" y2="5.08" width="0.1524" layer="91"/>
+<label x="10.16" y="5.08" size="1.778" layer="95"/>
+</segment>
+<segment>
+<pinref part="PACK+" gate="A" pin="SNS"/>
+<wire x1="40.64" y1="33.02" x2="91.44" y2="33.02" width="0.1524" layer="91"/>
+<wire x1="91.44" y1="45.72" x2="86.36" y2="45.72" width="0.1524" layer="91"/>
+<wire x1="86.36" y1="45.72" x2="81.28" y2="45.72" width="0.1524" layer="91"/>
+<wire x1="81.28" y1="45.72" x2="78.74" y2="45.72" width="0.1524" layer="91"/>
+<wire x1="91.44" y1="33.02" x2="91.44" y2="45.72" width="0.1524" layer="91"/>
+<junction x="91.44" y="45.72"/>
+<pinref part="L3" gate="G$1" pin="2"/>
+<pinref part="C6" gate="G$1" pin="1"/>
+<junction x="81.28" y="45.72"/>
+<label x="86.36" y="45.72" size="1.778" layer="95"/>
+<pinref part="C8" gate="G$1" pin="1"/>
+<junction x="86.36" y="45.72"/>
+</segment>
+</net>
